Commit message: changed to real dimensions+friction to wheels

File: taller1/urdf/robot.xacro (robot description, xacro)
@@ -11,5 +11,5 @@
         <origin xyz="0.0 0 0.0" rpy="0 0 $(eval pi/4*0)"/>
         <geometry>
-          <cylinder radius="0.3" length="0.10"/>
+          <cylinder radius="0.15" length="0.05"/>
         </geometry>
         <material name="blueish">
@@ -32,5 +32,5 @@
         <origin xyz="0.0 0 0.0" rpy="0 0 $(eval pi/4*0)"/>
         <geometry>
-          <cylinder radius="0.033" length="0.03"/>
+          <cylinder radius="0.025" length="0.03"/>
         </geometry>
         <material name="grisish">
@@ -41,5 +41,5 @@
       <origin xyz="0.0 0 0.0" rpy="0 0 0"/>
       <geometry>
-        <cylinder radius="0.033" length="0.03"/>
+        <cylinder radius="0.025" length="0.03"/>
       </geometry>
     </collision>
@@ -53,5 +53,5 @@
       <origin xyz="0.0 0 0.0" rpy="0 0 0"/>
       <geometry>
-        <cylinder radius="0.033" length="0.03"/>
+        <cylinder radius="0.025" length="0.03"/>
       </geometry>
       <material name="grisish">
@@ -62,5 +62,5 @@
     <origin xyz="0.0 0 0.0" rpy="0 0 0"/>
     <geometry>
-      <cylinder radius="0.033" length="0.03"/>
+      <cylinder radius="0.025" length="0.03"/>
     </geometry>
   </collision>
@@ -74,5 +74,5 @@
       <origin xyz="0.0 0 0.0" rpy="0 0 0"/>
       <geometry>
-        <sphere radius="0.033"/>
+        <sphere radius="0.025"/>
       </geometry>
       <material name="grisish">
@@ -83,5 +83,5 @@
     <origin xyz="0.0 0 0.0" rpy="0 0 0"/>
     <geometry>
-      <sphere radius="0.033"/>
+      <sphere radius="0.025"/>
     </geometry>
   </collision>
@@ -95,5 +95,5 @@
       <origin xyz="0.0 0 0.0" rpy="0 0 0"/>
       <geometry>
-        <sphere radius="0.033"/>
+        <sphere radius="0.025"/>
       </geometry>
       <material name="grisish">
@@ -104,5 +104,5 @@
     <origin xyz="0.0 0 0.0" rpy="0 0 0"/>
     <geometry>
-      <sphere radius="0.033"/>
+      <sphere radius="0.025"/>
     </geometry>
   </collision>

File: taller1/urdf/robot_joints.xacro (robot description, xacro)
@@ -12,5 +12,5 @@
 		<child link="wheel_left"/>
 		<axis xyz="0 0 1" rpy="0 0 0" />
-		<origin xyz="0.0 0.2 0.0" rpy="$(eval pi/2) 0 $(eval pi)"/>
+		<origin xyz="0.0 0.12 0.0" rpy="$(eval pi/2) 0 $(eval pi)"/>
 	</joint>
 	<joint name="wheel_rigth_joint" type="continuous">
@@ -18,5 +18,5 @@
 		<child link="wheel_rigth"/>
 		<axis xyz="0 0 1" rpy="0 0 0" />
-		<origin xyz="0.0 -0.2 0.0" rpy="$(eval pi/2) 0 $(eval pi)"/>
+		<origin xyz="0.0 -0.12 0.0" rpy="$(eval pi/2) 0 $(eval pi)"/>
 	</joint>
 	<joint name="pivot_back_joint" type="continuous">
@@ -24,5 +24,5 @@
 		<child link="pivot_back"/>
 		<axis xyz="0 0 1" rpy="0 0 0" />
-		<origin xyz="-0.2 0.0 0.0" rpy="$(eval pi/2) 0 0"/>
+		<origin xyz="-0.12 0.0 0.0" rpy="$(eval pi/2) 0 0"/>
 	</joint>
 	<joint name="pivot_front_joint" type="continuous">
@@ -30,5 +30,5 @@
 		<child link="pivot_front"/>
 		<axis xyz="0 0 1" rpy="0 0 0" />
-		<origin xyz="0.2 0.0 0.0" rpy="$(eval pi/2) 0 0"/>
+		<origin xyz="0.12 0.0 0.0" rpy="$(eval pi/2) 0 0"/>
 	</joint>
 </robot>

Commit message: corrected model collision

File: taller1/urdf/robot.xacro (robot description, xacro)
@@ -20,5 +20,5 @@
       <origin xyz="0.0 0 0.0" rpy="0 0 $(eval pi/4*0)"/>
       <geometry>
-        <cylinder radius="0.3" length="0.10"/>
+        <cylinder radius="0.15" length="0.10"/>
       </geometry>
     </collision>

Commit message: added geomerty for direction visualization

File: taller1/urdf/robot.xacro (robot description, xacro)
@@ -27,4 +27,22 @@
         <inertia ixx="0.01" iyy="0.01" izz="0.01" ixy="0.0" ixz="0.0" iyz="0.0" />
     </inertial>
+    <visual name="flecha">
+        <origin xyz="0.0 -0.05 0.03" rpy="0 1.57 $(eval pi/6)"/>
+        <geometry>
+          <cylinder radius="0.02" length="0.2"/>
+        </geometry>
+        <material name="black">
+          <color rgba="0.0 0.0 0.0 1.0"/>
+        </material>
+    </visual>
+    <visual name="flecha">
+        <origin xyz="0.0 0.05 0.03" rpy="0 1.57 $(eval -pi/6)"/>
+        <geometry>
+          <cylinder radius="0.02" length="0.2"/>
+        </geometry>
+        <material name="black">
+          <color rgba="0.0 0.0 0.0 1.0"/>
+        </material>
+    </visual>
   </link>
   <link name="wheel_left">
