Commit message: some small changes and additions

File: final_project/kmr_iiwa/urdf/arm/iiwa_joints.xacro (robot description, xacro)
@@ -3,21 +3,4 @@
  	<!--Joints-->
 	<!--joint1-->
-	<!-- <joint name="joint_1" type="revolute">
-    <origin rpy="0 0 0" xyz="0 0 0.3"/>
-    <parent link="base_arm"/>
-    <child link="link1"/>
-    <axis xyz="0 0 1"/>
-    <limit effort="1000" lower="-3.1416" upper="3.1416" velocity="2.618"/>
-  </joint>
-  <transmission name="trans_joint_1">
-		<type>transmission_interface/SimpleTransmission</type>
-		<joint name="joint_1">
-			<hardwareInterface>hardware_interface/PositionJointInterface</hardwareInterface>
-		</joint>
-		<actuator name="motor_joint_1">
-			<hardwareInterface>hardware_interface/PositionJointInterface</hardwareInterface>
-			<mechanicalReduction>1</mechanicalReduction>
-		</actuator>
-  </transmission> -->
 	<joint name="joint_a1" type="revolute">
 			<origin xyz="0 0 0.17" rpy="0 0 0"/>

File: final_project/kmr_iiwa/urdf/mobile_base/kmr.xacro (robot description, xacro)
@@ -56,5 +56,5 @@
       </geometry>
     </collision>
-    <visual name="mid_base">
+    <!-- <visual name="mid_base">
       <origin rpy="0 0 0" xyz="0 0 -0.2865"/>
       <geometry>
@@ -68,6 +68,6 @@
         <box size="0.920 0.51 0.055"/>
       </geometry>
-    </collision>
-    <visual name="bottom_base">
+    </collision> -->
+    <!-- <visual name="bottom_base">
       <origin rpy="0 0 0" xyz="0 0 -0.353"/>
       <geometry>
@@ -81,5 +81,5 @@
         <box size="1.08 0.63 0.085"/>
       </geometry>
-    </collision>
+    </collision> -->
     <inertial>
       <mass value="339.96"/>
